File: Hardware/PCB-uri/pcb4_placa_retea_v1/pcb4_placa_retea_v1.kicad_sch (KiCad schematic)
At the start: 62 parts, among them J1 Conn_01x10_Pin, J10 Screw_Terminal_01x02, J5 Screw_Terminal_01x02, J6 Screw_Terminal_01x02, J7 Screw_Terminal_01x02, J8 Screw_Terminal_01x02, J9 Screw_Terminal_01x02, U1 ISO7721D, U10 THVD1450D, U2 ISO7721D, U3 ISO7721D, U4 B0505S-1WR2, U5 THVD1450D, U6 THVD1450D, U7 THVD1450D, U8 THVD1450D, U9 THVD1450D

Commit message: Am mai lucrat la placa de retea sa intre intr-un dreptunghi de 100x75 si am mai lucrat putin la trasee (le-am facut de 0.5, ca sa stiu o treaba. Nu stiu cat de corect este, doar ca sunt constrans si de procedeul de gravare de acasa care este unul imperfect). Am dat comanda de piese, trebuie sa ajunga saptamana ce vine. Acum bag mare pe partea de software si ce am zis in mesajul anterior.
Parts:
- added C16: 100nF, symbol Device:C
Connections:
- net at C10.1, C11.1, C12.1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: now also C16.1
- net at C10.2, C11.2, C12.2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: now also C16.2
Changed lines of the file:
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@@
 	)
 	(junction
+		(at 226.06 81.28)
+		(diameter 0)
+		(color 0 0 0 0)
+	)
+	(junction
 		(at 86.36 139.7)
 		(diameter 0)
@@
 	)
 	(junction
+		(at 226.06 88.9)
+		(diameter 0)
+		(color 0 0 0 0)
+	)
+	(junction
 		(at 24.13 93.98)
 		(diameter 0)
@@
 	(wire
 		(pts
+			(xy 226.06 88.9) (xy 228.6 88.9)
+		)
+		(stroke
+			(width 0)
+			(type default)
+		)
+	)
+	(wire
+		(pts
 			(xy 118.11 78.74) (xy 118.11 81.28)
 		)
@@
 	(wire
 		(pts
-			(xy 209.55 88.9) (xy 228.6 88.9)
+			(xy 209.55 88.9) (xy 226.06 88.9)
 		)
 		(stroke
@@
 	(wire
 		(pts
-			(xy 220.98 81.28) (xy 232.41 81.28)
+			(xy 220.98 81.28) (xy 226.06 81.28)
 		)
 		(stroke
@@
 	(wire
 		(pts
+			(xy 226.06 81.28) (xy 232.41 81.28)
+		)
+		(stroke
+			(width 0)
+			(type default)
+		)
+	)
+	(wire
+		(pts
 			(xy 58.42 93.98) (xy 62.23 93.98)
 		)
@@
 					(unit 1)
 				)
+			)
+		)
+	)
+	(symbol
+		(lib_id "Device:C")
+		(at 226.06 85.09 0)
+		(unit 1)
+		(body_style 1)
+		(exclude_from_sim no)
+		(in_bom yes)
+		(on_board yes)
+		(in_pos_files yes)
+		(dnp no)
+		(fields_autoplaced yes)
+		(property "Reference" "C16"
+			(at 229.87 83.8199 0)
+			(show_name no)
+			(do_not_autoplace no)
+			(effects
+				(font
+					(size 1.27 1.27)
+				)
+				(justify left)
+			)
+		)
+		(property "Value" "100nF"
+			(at 229.87 86.3599 0)
+			(show_name no)
+			(do_not_autoplace no)
+			(effects
+				(font
+					(size 1.27 1.27)
+				)
+				(justify left)
+			)
+		)
+		(property "Footprint" ""
+			(at 227.0252 88.9 0)
+			(hide yes)
+			(show_name no)
+			(do_not_autoplace no)
+			(effects
+				(font
+					(size 1.27 1.27)
+				)
+			)
+		)
+		(property "Datasheet" ""
+			(at 226.06 85.09 0)
+			(hide yes)
+			(show_name no)
+			(do_not_autoplace no)
+			(effects
+				(font
+					(size 1.27 1.27)
+				)
+			)
+		)
+		(property "Description" "Unpolarized capacitor"
+			(at 226.06 85.09 0)
+			(hide yes)
+			(show_name no)
+			(do_not_autoplace no)
+			(effects
+				(font
+					(size 1.27 1.27)
+				)
+			)
+		)
+		(pin "2"
+		)
+		(pin "1"
+		)
+		(instances
+			(project "pcb4_placa_retea_v1"
+				(path "/e8f57aa6-9eec-405a-bc1f-aa1310f29cd4"
+					(reference "C16")
+					(unit 1)
+				)
