File: Dezvoltare_Proiect/Hardware/PCB-uri/Carduri_retea/Carduri_retea.kicad_pcb (KiCad board)
At the start: 2 copper layers, 60 parts, among them J1 Conn_01x03_Pin, J17 Screw_Terminal_01x02, J18 Screw_Terminal_01x02, J19 Conn_01x04_Pin, J2 Conn_01x03_Pin, J22 Conn_01x04_Pin, J25 Screw_Terminal_01x02, J26 Screw_Terminal_01x02, J37 Screw_Terminal_01x02, J38 Conn_01x04_Pin, J39 Screw_Terminal_01x02, J4 Conn_01x03_Pin, U10 THVD1450D, U11 THVD1450D, U13 ISO7721DWV, U14 ISO7721DWV, U15 ISO7721DWV, U16 THVD1450D, U7 THVD1450D, U8 THVD1450D, U9 THVD1450D

Commit message: Actualizare PCB-uri, componente custom, acces la documentatia de pe overleaf.
Parts:
- added C10: 100nF, Capacitor_SMD:C_0805_2012Metric, F.Cu at (183.4, 96.5)
- added C10: 100nF, Capacitor_SMD:C_0805_2012Metric, F.Cu at (116.5, 96.5)
- added C11: 100nF, Capacitor_SMD:C_0805_2012Metric, F.Cu at (187.0, 86.0)
- added C11: 100nF, Capacitor_SMD:C_0805_2012Metric, F.Cu at (120.0, 86.0)
- added C2: 100nF, Capacitor_SMD:C_0805_2012Metric, F.Cu at (201.5, 81.0)
- added C2: 100nF, Capacitor_SMD:C_0805_2012Metric, F.Cu at (134.5, 81.0)
- added C22: 100nF, Capacitor_SMD:C_0805_2012Metric, F.Cu at (205.0, 27.4)
- added C22: 100nF, Capacitor_SMD:C_0805_2012Metric, F.Cu at (274.0, 27.4)
- added C22: 100nF, Capacitor_SMD:C_0805_2012Metric, F.Cu at (136.5, 27.4)
- added C23: 100nF, Capacitor_SMD:C_0805_2012Metric, F.Cu at (191.0, 32.5)
- added C23: 100nF, Capacitor_SMD:C_0805_2012Metric, F.Cu at (260.0, 32.5)
- added C23: 100nF, Capacitor_SMD:C_0805_2012Metric, F.Cu at (122.5, 32.5)
- added C24: 100nF, Capacitor_SMD:C_0805_2012Metric, F.Cu at (118.5, 43.0)
- added C24: 100nF, Capacitor_SMD:C_0805_2012Metric, F.Cu at (187.1, 43.0)
- added C24: 100nF, Capacitor_SMD:C_0805_2012Metric, F.Cu at (256.1, 43.0)
- added C5: 100nF, Capacitor_SMD:C_0805_2012Metric, F.Cu at (183.4, 75.5)
- added C5: 100nF, Capacitor_SMD:C_0805_2012Metric, F.Cu at (116.5, 75.5)
- added C9: 100nF, Capacitor_SMD:C_0805_2012Metric, F.Cu at (256.1, 22.0)
- added C9: 100nF, Capacitor_SMD:C_0805_2012Metric, F.Cu at (187.1, 22.0)
- added C9: 100nF, Capacitor_SMD:C_0805_2012Metric, F.Cu at (118.5, 22.0)
- added D2: SM712_SOT23, Package_TO_SOT_SMD:SOT-23, F.Cu at (174.6, 80.0)
- added D2: SM712_SOT23, Package_TO_SOT_SMD:SOT-23, F.Cu at (107.6, 80.0)
- added D3: SM712_SOT23, Package_TO_SOT_SMD:SOT-23, F.Cu at (174.6, 91.5)
- added D3: SM712_SOT23, Package_TO_SOT_SMD:SOT-23, F.Cu at (107.6, 91.5)
- added D7: SM712_SOT23, Package_TO_SOT_SMD:SOT-23, F.Cu at (109.6, 26.4)
- added D7: SM712_SOT23, Package_TO_SOT_SMD:SOT-23, F.Cu at (247.1, 26.4)
- added D7: SM712_SOT23, Package_TO_SOT_SMD:SOT-23, F.Cu at (178.1, 26.4)
- added D8: SM712_SOT23, Package_TO_SOT_SMD:SOT-23, F.Cu at (247.1, 38.5)
- added D8: SM712_SOT23, Package_TO_SOT_SMD:SOT-23, F.Cu at (109.6, 38.5)
- added D8: SM712_SOT23, Package_TO_SOT_SMD:SOT-23, F.Cu at (178.1, 38.5)
- added J1: Conn_01x03_Pin, Connector_PinHeader_2.54mm:PinHeader_1x03_P2.54mm_Vertical, F.Cu at (179.5, 32.5)
- added J1: Conn_01x03_Pin, Connector_PinHeader_2.54mm:PinHeader_1x03_P2.54mm_Vertical, F.Cu at (248.5, 32.5)
- added J1: Conn_01x03_Pin, Connector_PinHeader_2.54mm:PinHeader_1x03_P2.54mm_Vertical, F.Cu at (111.0, 32.5)
- added J17: Screw_Terminal_01x02, TerminalBlock:TerminalBlock_MaiXu_MX126-5.0-02P_1x02_P5.00mm, F.Cu at (95.5, 77.8)
- added J17: Screw_Terminal_01x02, TerminalBlock:TerminalBlock_MaiXu_MX126-5.0-02P_1x02_P5.00mm, F.Cu at (162.5, 77.8)
- added J18: Screw_Terminal_01x02, TerminalBlock:TerminalBlock_MaiXu_MX126-5.0-02P_1x02_P5.00mm, F.Cu at (95.5, 89.8)
- added J18: Screw_Terminal_01x02, TerminalBlock:TerminalBlock_MaiXu_MX126-5.0-02P_1x02_P5.00mm, F.Cu at (162.5, 89.8)
- added J19: Conn_01x04_Pin, Connector_PinHeader_2.54mm:PinHeader_1x04_P2.54mm_Vertical, F.Cu at (205.0, 82.0)
- added J19: Conn_01x04_Pin, Connector_PinHeader_2.54mm:PinHeader_1x04_P2.54mm_Vertical, F.Cu at (138.0, 82.0)
- added J37: Screw_Terminal_01x02, TerminalBlock:TerminalBlock_MaiXu_MX126-5.0-02P_1x02_P5.00mm, F.Cu at (235.0, 24.2)
- added J37: Screw_Terminal_01x02, TerminalBlock:TerminalBlock_MaiXu_MX126-5.0-02P_1x02_P5.00mm, F.Cu at (97.5, 24.2)
- added J37: Screw_Terminal_01x02, TerminalBlock:TerminalBlock_MaiXu_MX126-5.0-02P_1x02_P5.00mm, F.Cu at (166.0, 24.2)
- added J38: Conn_01x04_Pin, Connector_PinHeader_2.54mm:PinHeader_1x04_P2.54mm_Vertical, F.Cu at (208.5, 28.5)
- added J38: Conn_01x04_Pin, Connector_PinHeader_2.54mm:PinHeader_1x04_P2.54mm_Vertical, F.Cu at (140.0, 28.5)
- added J38: Conn_01x04_Pin, Connector_PinHeader_2.54mm:PinHeader_1x04_P2.54mm_Vertical, F.Cu at (277.5, 28.5)
- added J39: Screw_Terminal_01x02, TerminalBlock:TerminalBlock_MaiXu_MX126-5.0-02P_1x02_P5.00mm, F.Cu at (235.0, 36.2)
- added J39: Screw_Terminal_01x02, TerminalBlock:TerminalBlock_MaiXu_MX126-5.0-02P_1x02_P5.00mm, F.Cu at (97.5, 36.2)
- added J39: Screw_Terminal_01x02, TerminalBlock:TerminalBlock_MaiXu_MX126-5.0-02P_1x02_P5.00mm, F.Cu at (166.0, 36.2)
- added J4: Conn_01x03_Pin, Connector_PinHeader_2.54mm:PinHeader_1x03_P2.54mm_Vertical, F.Cu at (176.0, 86.0)
- added J4: Conn_01x03_Pin, Connector_PinHeader_2.54mm:PinHeader_1x03_P2.54mm_Vertical, F.Cu at (109.0, 86.0)
- added R11: 10k, Resistor_SMD:R_0805_2012Metric, F.Cu at (259.9, 22.0)
- added R11: 10k, Resistor_SMD:R_0805_2012Metric, F.Cu at (190.9, 22.0)
- added R11: 10k, Resistor_SMD:R_0805_2012Metric, F.Cu at (122.4, 22.0)
- added R12: 120Ω, Resistor_SMD:R_0805_2012Metric, F.Cu at (251.5, 38.4)
- added R12: 120Ω, Resistor_SMD:R_0805_2012Metric, F.Cu at (114.0, 38.4)
- added R12: 120Ω, Resistor_SMD:R_0805_2012Metric, F.Cu at (182.5, 38.4)
- added R3: 120Ω, Resistor_SMD:R_0805_2012Metric, F.Cu at (112.0, 79.9)
- added R3: 120Ω, Resistor_SMD:R_0805_2012Metric, F.Cu at (179.0, 79.9)
- added R4: 120Ω, Resistor_SMD:R_0805_2012Metric, F.Cu at (179.0, 91.4)
- added R4: 120Ω, Resistor_SMD:R_0805_2012Metric, F.Cu at (112.0, 91.4)
- added R7: 120Ω, Resistor_SMD:R_0805_2012Metric, F.Cu at (114.0, 26.4)
- added R7: 120Ω, Resistor_SMD:R_0805_2012Metric, F.Cu at (251.5, 26.4)
- added R7: 120Ω, Resistor_SMD:R_0805_2012Metric, F.Cu at (182.5, 26.4)
- added R9: 10k, Resistor_SMD:R_0805_2012Metric, F.Cu at (187.6, 75.5)
- added R9: 10k, Resistor_SMD:R_0805_2012Metric, F.Cu at (120.6, 75.5)
- added TH13: Thermistor_PTC, Resistor_SMD:R_0805_2012Metric, F.Cu at (105.9, 29.5)
- added TH13: Thermistor_PTC, Resistor_SMD:R_0805_2012Metric, F.Cu at (174.4, 29.5)
- added TH13: Thermistor_PTC, Resistor_SMD:R_0805_2012Metric, F.Cu at (243.4, 29.5)
- added TH14: Thermistor_PTC, Resistor_SMD:R_0805_2012Metric, F.Cu at (243.4, 24.0)
- added TH14: Thermistor_PTC, Resistor_SMD:R_0805_2012Metric, F.Cu at (105.9, 24.0)
- added TH14: Thermistor_PTC, Resistor_SMD:R_0805_2012Metric, F.Cu at (174.4, 24.0)
- added TH15: Thermistor_PTC, Resistor_SMD:R_0805_2012Metric, F.Cu at (105.9, 41.0)
- added TH15: Thermistor_PTC, Resistor_SMD:R_0805_2012Metric, F.Cu at (174.4, 41.0)
- added TH15: Thermistor_PTC, Resistor_SMD:R_0805_2012Metric, F.Cu at (243.4, 41.0)
- added TH16: Thermistor_PTC, Resistor_SMD:R_0805_2012Metric, F.Cu at (174.4, 35.5)
- added TH16: Thermistor_PTC, Resistor_SMD:R_0805_2012Metric, F.Cu at (243.4, 35.5)
- added TH16: Thermistor_PTC, Resistor_SMD:R_0805_2012Metric, F.Cu at (105.9, 35.5)
- added TH5: Thermistor_PTC, Resistor_SMD:R_0805_2012Metric, F.Cu at (170.9, 83.0)
- added TH5: Thermistor_PTC, Resistor_SMD:R_0805_2012Metric, F.Cu at (103.9, 83.0)
- added TH6: Thermistor_PTC, Resistor_SMD:R_0805_2012Metric, F.Cu at (170.9, 77.5)
- added TH6: Thermistor_PTC, Resistor_SMD:R_0805_2012Metric, F.Cu at (103.9, 77.5)
- added TH7: Thermistor_PTC, Resistor_SMD:R_0805_2012Metric, F.Cu at (103.9, 94.5)
- added TH7: Thermistor_PTC, Resistor_SMD:R_0805_2012Metric, F.Cu at (170.9, 94.5)
- added TH8: Thermistor_PTC, Resistor_SMD:R_0805_2012Metric, F.Cu at (170.9, 89.0)
- added TH8: Thermistor_PTC, Resistor_SMD:R_0805_2012Metric, F.Cu at (103.9, 89.0)
- added U11: THVD1450D, Package_SO:SOIC-8_3.9x4.9mm_P1.27mm, F.Cu at (258.0, 26.4)
- added U11: THVD1450D, Package_SO:SOIC-8_3.9x4.9mm_P1.27mm, F.Cu at (120.5, 26.4)
- added U11: THVD1450D, Package_SO:SOIC-8_3.9x4.9mm_P1.27mm, F.Cu at (189.0, 26.4)
- added U13: ISO7721DWV, Package_SO:SOIC-8_7.5x5.85mm_P1.27mm, F.Cu at (196.0, 86.0)
- added U13: ISO7721DWV, Package_SO:SOIC-8_7.5x5.85mm_P1.27mm, F.Cu at (129.0, 86.0)
- added U15: ISO7721DWV, Package_SO:SOIC-8_7.5x5.85mm_P1.27mm, F.Cu at (268.7, 32.6)
- added U15: ISO7721DWV, Package_SO:SOIC-8_7.5x5.85mm_P1.27mm, F.Cu at (199.7, 32.6)
- added U15: ISO7721DWV, Package_SO:SOIC-8_7.5x5.85mm_P1.27mm, F.Cu at (131.2, 32.6)
- added U16: THVD1450D, Package_SO:SOIC-8_3.9x4.9mm_P1.27mm, F.Cu at (189.0, 38.4)
- added U16: THVD1450D, Package_SO:SOIC-8_3.9x4.9mm_P1.27mm, F.Cu at (258.0, 38.4)
- added U16: THVD1450D, Package_SO:SOIC-8_3.9x4.9mm_P1.27mm, F.Cu at (120.5, 38.4)
- added U7: THVD1450D, Package_SO:SOIC-8_3.9x4.9mm_P1.27mm, F.Cu at (118.5, 79.9)
- added U7: THVD1450D, Package_SO:SOIC-8_3.9x4.9mm_P1.27mm, F.Cu at (185.5, 79.9)
- added U8: THVD1450D, Package_SO:SOIC-8_3.9x4.9mm_P1.27mm, F.Cu at (118.5, 91.9)
- added U8: THVD1450D, Package_SO:SOIC-8_3.9x4.9mm_P1.27mm, F.Cu at (185.5, 91.9)
Routing:
- net Net-(D7-common): track 73.5 -> 294.1 mm, vias 6 -> 24
- net Net-(D2-common): track 70.6 -> 211.9 mm, vias 6 -> 18
- net Net-(J1-Pin_2): track 45.2 -> 181.0 mm, vias 3 -> 12
- net Net-(J4-Pin_2): track 44.4 -> 133.3 mm, vias 3 -> 9
- net Net-(J1-Pin_3): track 15.0 -> 59.8 mm, vias 3 -> 12
- net Net-(J38-Pin_2): track 14.7 -> 58.9 mm, vias 3 -> 12
- net Net-(D7-A1): track 12.2 -> 48.8 mm
- net Net-(D8-A2): track 12.1 -> 48.5 mm
- net Net-(D8-A1): track 12.0 -> 47.9 mm
- net Net-(D7-A2): track 11.9 -> 47.6 mm
- net Net-(J19-Pin_2): track 14.9 -> 44.8 mm, vias 3 -> 9
- net Net-(D2-A1): track 12.2 -> 36.7 mm
- net Net-(D3-A1): track 12.2 -> 36.6 mm
- net Net-(D3-A2): track 12.2 -> 36.5 mm
- net Net-(D2-A2): track 12.0 -> 36.0 mm
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Other:
- board outline added: 256 x 133.5 mm
- board text added: "Cartela date in sync out"
- board text added: "Cartela date in sync out (nod central)"
- board text added: "Cartela date out sync in"
