File: Dezvoltare_Proiect/Hardware/PCB-uri/Placa_retea_si_carduri/Placa_retea_si_carduri.kicad_pcb (KiCad board)
At the start: 2 copper layers, 29 parts, among them J1 Conn_01x03_Socket, J2 Conn_01x03_Socket, J28 Conn_01x04_Socket, J29 Conn_01x04_Socket, J3 Conn_01x03_Socket, J30 Conn_01x08_Pin, J31 Conn_01x08_Pin, J32 Conn_01x04_Socket, J33 Conn_01x04_Socket, J34 Conn_01x04_Socket, J35 Conn_01x04_Socket, J36 Conn_01x04_Socket, J4 Conn_01x03_Socket, J5 Conn_01x03_Socket, J6 Conn_01x03_Socket, J7 Conn_01x03_Socket, J8 Conn_01x02_Pin, U2 1769405141, U3 1769405141

Commit message: Incarc ce am mai lucrat in ultima luna!
Other:
- board outline added: 238.5 x 152 mm

Commit message: Actualizare PCB-uri, componente custom, acces la documentatia de pe overleaf.
Parts:
- added C18: 4.7/10 uF, Capacitor_SMD:C_0805_2012Metric, B.Cu at (-30.0, 31.9)
- added C18: 4.7/10 uF, Capacitor_SMD:C_0805_2012Metric, B.Cu at (-34.0, 127.0)
- added C18: 4.7/10 uF, Capacitor_SMD:C_0805_2012Metric, B.Cu at (-31.0, -55.0)
- added C19: 1nF 2kV, Capacitor_THT:C_Disc_D8.0mm_W5.0mm_P7.50mm, F.Cu at (-14.0, 134.8)
- added C19: 1nF 2kV, Capacitor_THT:C_Disc_D8.0mm_W5.0mm_P7.50mm, F.Cu at (-10.0, 39.8)
- added C19: 1nF 2kV, Capacitor_THT:C_Disc_D8.0mm_W5.0mm_P7.50mm, F.Cu at (-11.0, -47.2)
- added C20: 4.7/10uF, Capacitor_SMD:C_0805_2012Metric, F.Cu at (-38.5, 43.0)
- added C20: 4.7/10uF, Capacitor_SMD:C_0805_2012Metric, F.Cu at (-39.5, -44.0)
- added C20: 4.7/10uF, Capacitor_SMD:C_0805_2012Metric, F.Cu at (-42.5, 138.0)
- added C21: 100nF, Capacitor_SMD:C_0805_2012Metric, F.Cu at (-42.5, 145.5)
- added C21: 100nF, Capacitor_SMD:C_0805_2012Metric, F.Cu at (-39.5, -36.5)
- added C21: 100nF, Capacitor_SMD:C_0805_2012Metric, F.Cu at (-38.5, 50.5)
- added FB2: 4.7/10 uH, Inductor_SMD:L_0805_2012Metric, F.Cu at (-40.5, -40.4)
- added FB2: 4.7/10 uH, Inductor_SMD:L_0805_2012Metric, F.Cu at (-39.5, 46.6)
- added FB2: 4.7/10 uH, Inductor_SMD:L_0805_2012Metric, F.Cu at (-43.5, 141.6)
- added J1: Conn_01x03_Socket, Connector_PinHeader_2.54mm:PinHeader_1x03_P2.54mm_Vertical, F.Cu at (-83.5, 54.6)
- added J1: Conn_01x03_Socket, Connector_PinHeader_2.54mm:PinHeader_1x03_P2.54mm_Vertical, F.Cu at (-84.5, -32.4)
- added J1: Conn_01x03_Socket, Connector_PinHeader_2.54mm:PinHeader_1x03_P2.54mm_Vertical, F.Cu at (-87.5, 149.6)
- added J2: Conn_01x03_Socket, Connector_PinHeader_2.54mm:PinHeader_1x03_P2.54mm_Vertical, F.Cu at (-53.5, 54.6)
- added J2: Conn_01x03_Socket, Connector_PinHeader_2.54mm:PinHeader_1x03_P2.54mm_Vertical, F.Cu at (-57.5, 149.6)
- added J2: Conn_01x03_Socket, Connector_PinHeader_2.54mm:PinHeader_1x03_P2.54mm_Vertical, F.Cu at (-54.5, -32.4)
- added J28: Conn_01x04_Socket, Connector_PinHeader_2.54mm:PinHeader_1x04_P2.54mm_Vertical, F.Cu at (-88.3, -61.5)
- added J28: Conn_01x04_Socket, Connector_PinHeader_2.54mm:PinHeader_1x04_P2.54mm_Vertical, F.Cu at (-91.3, 120.5)
- added J28: Conn_01x04_Socket, Connector_PinHeader_2.54mm:PinHeader_1x04_P2.54mm_Vertical, F.Cu at (-87.3, 25.5)
- added J3: Conn_01x03_Socket, Connector_PinHeader_2.54mm:PinHeader_1x03_P2.54mm_Vertical, F.Cu at (-27.5, 149.6)
- added J3: Conn_01x03_Socket, Connector_PinHeader_2.54mm:PinHeader_1x03_P2.54mm_Vertical, F.Cu at (-23.5, 54.6)
- added J3: Conn_01x03_Socket, Connector_PinHeader_2.54mm:PinHeader_1x03_P2.54mm_Vertical, F.Cu at (-24.5, -32.4)
- added J30: Conn_01x08_Pin, Connector_PinHeader_2.54mm:PinHeader_1x08_P2.54mm_Vertical, F.Cu at (-48.5, 110.5)
- added J30: Conn_01x08_Pin, Connector_PinHeader_2.54mm:PinHeader_1x08_P2.54mm_Vertical, F.Cu at (-45.5, -71.5)
- added J30: Conn_01x08_Pin, Connector_PinHeader_2.54mm:PinHeader_1x08_P2.54mm_Vertical, F.Cu at (-44.5, 15.5)
- added J32: Conn_01x04_Socket, Connector_PinHeader_2.54mm:PinHeader_1x04_P2.54mm_Vertical, F.Cu at (-58.1, -61.5)
- added J32: Conn_01x04_Socket, Connector_PinHeader_2.54mm:PinHeader_1x04_P2.54mm_Vertical, F.Cu at (-57.1, 25.5)
- added J32: Conn_01x04_Socket, Connector_PinHeader_2.54mm:PinHeader_1x04_P2.54mm_Vertical, F.Cu at (-61.1, 120.5)
- added J35: Conn_01x04_Socket, Connector_PinHeader_2.54mm:PinHeader_1x04_P2.54mm_Vertical, F.Cu at (-27.1, 25.5)
- added J35: Conn_01x04_Socket, Connector_PinHeader_2.54mm:PinHeader_1x04_P2.54mm_Vertical, F.Cu at (-31.1, 120.5)
- added J35: Conn_01x04_Socket, Connector_PinHeader_2.54mm:PinHeader_1x04_P2.54mm_Vertical, F.Cu at (-28.1, -61.5)
- added U2: 1769405141, Footprints:Wurth_1769405141_SMT-8, B.Cu at (-38.5, 34.5)
- added U2: 1769405141, Footprints:Wurth_1769405141_SMT-8, B.Cu at (-42.5, 129.5)
- added U2: 1769405141, Footprints:Wurth_1769405141_SMT-8, B.Cu at (-39.5, -52.5)
Routing:
- net Net-(J28-Pin_1): track 121.9 -> 487.5 mm, vias 6 -> 24
- net Net-(J1-Pin_1): track 104.7 -> 419.0 mm, vias 3 -> 12
- net Net-(J28-Pin_2): track 93.3 -> 373.1 mm, vias 3 -> 12
- net Net-(J1-Pin_2): track 63.9 -> 255.7 mm, vias 1 -> 4
- net Net-(J1-Pin_3): track 60.0 -> 240.0 mm
- net Net-(J30-Pin_4): track 41.0 -> 163.9 mm, vias 1 -> 4
- net Net-(J30-Pin_3): track 34.0 -> 136.1 mm, vias 3 -> 12
- net Net-(J28-Pin_3): track 28.4 -> 113.6 mm, vias 3 -> 12
- net Net-(J28-Pin_4): track 21.6 -> 86.4 mm, vias 1 -> 4
- net Net-(J30-Pin_6): track 15.8 -> 63.3 mm, vias 3 -> 12
- net Net-(J30-Pin_5): track 11.1 -> 44.3 mm, vias 1 -> 4
- net Net-(U2-+VOUT): track 8.75 -> 35.0 mm, vias 1 -> 4
Other:
- board size 238.5 x 152 mm -> 378.5 x 257 mm
